File: SolderPlate_Power/SolderPlate_Power.kicad_sch (KiCad schematic)
At the start: 22 parts, among them J1 N, J2 Fan, J2 LCD, J3 L, J4 SSR, J7 uCont, Q1 BSS138, Q2 BSS138, Q3 BSS138

Commit message: Added schematic PDFs
Other:
- title: (none) -> Solder Plate - Power Board
Changed lines of the file:
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@@
 (kicad_sch (version 20230121) (generator eeschema)
   (paper "A4")
+  (title_block
+    (title "Solder Plate - Power Board")
+    (rev "A")
+    (comment 1 "TiZed")
+  )
   (junction (at 264.795 34.925) (diameter 0) (color 0 0 0 0)
   )
